Commit message: 240222

File: URDFdir/BrandNewFlapper.urdf (robot description, URDF)
Before this commit: robot flapper, 5 links, 4 joints
Joints:
- removed joint left_Stroke_joint
- added joint left_stroke_joint: type continuous, parent torso, child left_wing_rod, origin xyz=0.016247 0 0.0095033 rpy=0 0 0, axis 0 0 1

File: URDFdir/flapper.urdf (robot description, URDF)
Before this commit: robot flapper, 5 links, 4 joints
Links:
- link left_wing: geometry collision mesh filename=./meshes/left_wing.STL; visual mesh filename=./meshes/left_wing.STL
- link left_wing_rod: geometry collision mesh filename=./meshes/left_wing_rod.STL; visual mesh filename=./meshes/left_wing_rod.STL
- link right_wing: geometry collision mesh filename=./meshes/right_wing.STL; visual mesh filename=./meshes/right_wing.STL
- link right_wing_rod: geometry collision mesh filename=./meshes/right_wing_rod.STL; visual mesh filename=./meshes/right_wing_rod.STL
- link torso: geometry collision mesh filename=./meshes/torso.STL; visual mesh filename=./meshes/torso.STL
Joints:
- removed joint left_Stroke_joint
- added joint left_stroke_joint: type continuous, parent torso, child left_wing_rod, origin xyz=0.016247 0 0.0095033 rpy=0 0 0, axis 0 0 1, limit lower=-1.57 upper=1.57 effort=0 velocity=0
- joint left_rotate_joint: limit lower=0 upper=0 effort=0 velocity=0 -> lower=-1.57 upper=1.57 effort=0 velocity=0; type revolute -> continuous
- joint right_rotate_joint: limit lower=0 upper=0 effort=0 velocity=0 -> lower=-1.57 upper=1.57 effort=0 velocity=0; type revolute -> continuous
- joint right_stroke_joint: limit lower=0 upper=0 effort=0 velocity=0 -> lower=-1.57 upper=1.57 effort=0 velocity=0; type revolute -> continuous
